File: mcp2221.kicad/mcp2221.sch (KiCad schematic (older format))
At the start: 26 parts, among them J1 Jumper 32 or 21, J2 Conn_01x04_Male, J3 Conn_01x03_Male, J4 Conn_01x06_Male, J5 Conn_01x03_Male, J6 Conn_01x06_Male, J7 Conn_01x02_Male, J8 Conn_01x02_Male, SW1 SW_Push, SW2 SW_Push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

Commit message: Rev 9: don't connect Vusb to 3.3V / changed R for LEDs to 150
Parts:
- R5, R6: value 1K -> 150
Connections:
- net 3.3V: no longer C2.1, U2.11 (VUSB)
- new net: C2.1, U2.11 (VUSB)
Other:
- note added: "VDD"
- moved on the sheet: C2
Changed lines of the file:
@@
 Sheet 1 1
 Title "MCP2221 Breakout"
-Date "2020-04-17"
-Rev "8"
+Date "2020-04-30"
+Rev "9"
 Comp "https://github.com/bablokb/pcb-mcp2221"
 Comment1 ""
@@
 U 1 1 5E4C2101
 P 4200 3150
-F 0 "R2" H 4270 3196 50  0000 L CNN
-F 1 "2.2k" H 4270 3105 50  0000 L CNN
+F 0 "R2" H 4250 3100 50  0000 L CNN
+F 1 "2.2k" H 4250 3000 50  0000 L CNN
 F 2 "user:R_1206_3216_Pad1.7x1.75mm_BB" V 4130 3150 50  0001 C CNN
 F 3 "~" H 4200 3150 50  0001 C CNN
@@
 U 1 1 5E4C2B00
 P 4450 3150
-F 0 "R1" H 4520 3196 50  0000 L CNN
-F 1 "2.2K" H 4520 3105 50  0000 L CNN
+F 0 "R1" H 4500 3100 50  0000 L CNN
+F 1 "2.2K" H 4500 3000 50  0000 L CNN
 F 2 "user:R_1206_3216_Pad1.7x1.75mm_BB" V 4380 3150 50  0001 C CNN
 F 3 "~" H 4450 3150 50  0001 C CNN
@@
 P 6650 4050
 F 0 "R5" H 6450 4100 50  0000 L CNN
-F 1 "1K" H 6450 4000 50  0000 L CNN
+F 1 "150" H 6450 4000 50  0000 L CNN
 F 2 "user:R_1206_3216_Pad1.7x1.75mm_BB" V 6580 4050 50  0001 C CNN
 F 3 "~" H 6650 4050 50  0001 C CNN
@@
 P 6900 4050
 F 0 "R6" H 6970 4096 50  0000 L CNN
-F 1 "1K" H 6970 4005 50  0000 L CNN
+F 1 "150" H 6970 4005 50  0000 L CNN
 F 2 "user:R_1206_3216_Pad1.7x1.75mm_BB" V 6830 4050 50  0001 C CNN
 F 3 "~" H 6900 4050 50  0001 C CNN
@@
 $EndComp
 $Comp
-L Device:C C2
-U 1 1 5E4DC43E
-P 3850 1050
-F 0 "C2" H 3600 1000 50  0000 C CNN
-F 1 "0.47µF" H 3550 1100 50  0000 C CNN
-F 2 "user:C_1206_3216_Pad1.7x1.75mm_BB" H 3888 900 50  0001 C CNN
-F 3 "~" H 3850 1050 50  0001 C CNN
-	1    3850 1050
-	-1   0    0    1
-$EndComp
-$Comp
 L power:GND #PWR03
 U 1 1 5E4DDCA8
-P 3850 900
-F 0 "#PWR03" H 3850 650 50  0001 C CNN
-F 1 "GND" V 3855 772 50  0000 R CNN
-F 2 "" H 3850 900 50  0001 C CNN
-F 3 "" H 3850 900 50  0001 C CNN
-	1    3850 900
-	-1   0    0    1
-$EndComp
-Wire Wire Line
-	4300 2500 4100 2500
+P 4300 1150
+F 0 "#PWR03" H 4300 900 50  0001 C CNN
+F 1 "GND" V 4305 1022 50  0000 R CNN
+F 2 "" H 4300 1150 50  0001 C CNN
+F 3 "" H 4300 1150 50  0001 C CNN
+	1    4300 1150
+	-1   0    0    1
+$EndComp
 $Comp
 L Connector:Conn_01x03_Male J1
@@
 P 3600 1900
 F 0 "J1" V 3662 2044 50  0000 L CNN
-F 1 "Jumper 32 or 21" V 3550 1700 50  0000 L CNN
+F 1 "Jumper 32 or 21" V 3950 1550 50  0000 L CNN
 F 2 "Connector_PinHeader_2.54mm:PinHeader_1x03_P2.54mm_Vertical" H 3600 1900 50  0001 C CNN
 F 3 "~" H 3600 1900 50  0001 C CNN
@@
 Wire Wire Line
 	3600 2150 4000 2150
-Wire Wire Line
-	4000 2150 4000 2450
 Connection ~ 4000 2600
-Wire Wire Line
-	4100 2500 4100 1450
-Wire Wire Line
-	3850 1450 3850 1200
-$Comp
-L power:GND #PWR04
-U 1 1 5E4E6294
-P 4300 1400
-F 0 "#PWR04" H 4300 1150 50  0001 C CNN
-F 1 "GND" V 4350 1550 50  0000 R CNN
-F 2 "" H 4300 1400 50  0001 C CNN
-F 3 "" H 4300 1400 50  0001 C CNN
-	1    4300 1400
-	0    1    1    0
-$EndComp
 $Comp
 L Device:R R3
@@
 Wire Wire Line
 	2300 1800 2300 1450
-Wire Wire Line
-	4100 1450 3850 1450
 Wire Wire Line
 	3450 1450 3550 1450
@@
 Wire Wire Line
 	8800 3400 8800 3050
-Connection ~ 3700 1450
-Connection ~ 3850 1450
-Wire Wire Line
-	3850 1450 3700 1450
 Connection ~ 8700 2500
 Wire Wire Line
@@
 Wire Wire Line
 	4000 2850 4000 3700
+Wire Wire Line
+	4000 2150 4000 2450
+$Comp
+L Device:C C2
+U 1 1 5E4DC43E
+P 4100 1350
+F 0 "C2" H 4150 1250 50  0000 C CNN
+F 1 "0.47µF" H 4050 1450 50  0000 C CNN
+F 2 "user:C_1206_3216_Pad1.7x1.75mm_BB" H 4138 1200 50  0001 C CNN
+F 3 "~" H 4100 1350 50  0001 C CNN
+	1    4100 1350
+	-1   0    0    1
+$EndComp
+Wire Wire Line
+	4100 2500 4300 2500
+Wire Wire Line
+	4300 1400 4300 1200
+Wire Wire Line
+	4100 1200 4300 1200
+Connection ~ 4300 1200
+Wire Wire Line
+	4300 1200 4300 1150
+Text Notes 4750 3800 0    50   ~ 0
+VDD
+Wire Wire Line
+	4100 1500 4100 2500
 $EndSCHEMATC

Commit message: Rev 10: fix order of D-/D+ in schematic+pcb
Connections:
- net USB-D+: now also USB1.3 (Pin_3); no longer USB1.4 (Pin_4)
- net USB-D-: now also USB1.4 (Pin_4); no longer USB1.3 (Pin_3)
Changed lines of the file:
@@
 Sheet 1 1
 Title "MCP2221 Breakout"
-Date "2020-04-30"
-Rev "9"
+Date "2020-05-01"
+Rev "10"
 Comp "https://github.com/bablokb/pcb-mcp2221"
 Comment1 ""
@@
 USB-D+
 Text Label 2300 2400 0    50   ~ 0
+USB-D+
+Text Label 2300 2300 0    50   ~ 0
 USB-D-
-Text Label 2300 2300 0    50   ~ 0
-USB-D+
 Text Label 4300 1700 2    50   ~ 0
 GP3
